Commit message: factory_robot1: move drive wheels +0.12 forward (wheelbase 0.25->0.37m) to kill start/stop pitch

File: src/fp_factory_sim/urdf/factory_robot1.xacro (robot description, xacro)
@@ -51,5 +51,5 @@
       <parent link="base_link"/>
       <child link="${prefix}_wheel_link"/>
-      <origin xyz="0 ${y_reflect*0.3} ${wheel_r}" rpy="${-pi/2} 0 0"/>
+      <origin xyz="0.12 ${y_reflect*0.3} ${wheel_r}" rpy="${-pi/2} 0 0"/>
       <axis xyz="0 0 1"/>
     </joint>
